File: KiCad/Splitty.kicad_sch (KiCad schematic)
At the start: 12 parts, among them J1 VIN (7V5 - 40VDC) 10A Max, J10 VOUT C1, J2 VOUT A1, J3 VOUT A2, J4 VOUT A3, J5 VOUT B1, J6 VOUT B2, J7 VOUT B3, J8 VOUT C3, J9 VOUT C2

Commit message: Update Splitty
Parts:
- added F1: 10A Max, symbol Device:Fuse
- added SW1: 10A, symbol Switch:SW_SPST
Connections:
- net at J10.1, J2.1, J3.1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: now also SW1.2 (B); no longer J1.1
- new net: F1.1, J1.1
- new net: F1.2, SW1.1 (A)
Other:
- moved on the sheet: J1, J10, J2, J3, J4, J5, J6, J7, J8, J9, TH1, U1
